Commit message: fix bug npc collision

File: resources/objects/sheep.urdf (robot description, URDF)
Before this commit: robot sheep, 7 links, 6 joints
Links:
- link body: mass 0.03 -> 5; geometry collision cylinder length=0.5 radius=0.25; visual sphere radius=0.2

Commit message: sheep bug no collision

File: resources/objects/sheep.urdf (robot description, URDF)
Before this commit: robot sheep, 7 links, 6 joints
Links:
- link FL_leg: geometry visual cylinder length=0.25 radius=0.03
- link FR_leg: geometry visual cylinder length=0.25 radius=0.03
- link RL_leg: geometry visual cylinder length=0.25 radius=0.03
- link RR_leg: geometry visual cylinder length=0.25 radius=0.03
- link body: geometry collision cylinder length=0.5 radius=0.2; visual sphere radius=0.2
- link face: geometry visual sphere radius=0.08
- link head: geometry visual sphere radius=0.08
