Commit message: update go1push

File: resources/objects/box.urdf (robot description, URDF)
Before this commit: robot box, 1 links, 0 joints
Links:
- link box: mass 10 -> 8

Commit message: add render

File: resources/objects/box.urdf (robot description, URDF)
Before this commit: robot box, 1 links, 0 joints
Links:
- link box: mass 8 -> 6
