Commit message: clip command to (-1,1)

File: resources/objects/seesaw.urdf (robot description, URDF)
Before this commit: robot sheep, 2 links, 1 joints
Links:
- link base: geometry collision box size=1 1 0.02; visual box size=1 1 0.02
- link seesaw: geometry collision box size=4.123 1 0.02; visual box size=4.123 1 0.02
Joints:
- joint link: origin xyz=-2.42 0 -0.45 rpy=0 0 0 -> xyz=-2.4 0 -0.46 rpy=0 0 0

Commit message: update sheep movement

File: resources/objects/seesaw.urdf (robot description, URDF)
Before this commit: robot sheep, 2 links, 1 joints
Links:
- added link column; collision cylinder length=1 radius=0.2; visual cylinder length=1 radius=0.15
Joints:
- added joint column_mount: type fixed, parent base, child column

Commit message: change sheep terrain

File: resources/objects/seesaw.urdf (robot description, URDF)
Before this commit: robot sheep, 3 links, 2 joints
Links:
- link base: geometry collision box size=1 1 0.03; visual box size=1 1 0.03
- link seesaw: geometry collision box size=4.123 1 0.03; visual box size=4.123 1 0.03
Joints:
- joint link: limit effort=33.5 velocity=28 -> effort=33.5 velocity=1; origin xyz=-2.4 0 -0.46 rpy=0 0 0 -> xyz=-2.4 0 -0.455 rpy=0 0 0

Commit message: update envs

File: resources/objects/seesaw.urdf (robot description, URDF)
Before this commit: robot sheep, 3 links, 2 joints
Links:
- link seesaw: mass 10 -> 100
Joints:
- joint link: limit effort=33.5 velocity=1 -> effort=0 velocity=0.2

Commit message: update docs 2023.3.24

File: resources/objects/seesaw.urdf (robot description, URDF)
Before this commit: robot sheep, 3 links, 2 joints
Links:
- added link shaft_l; visual cylinder length=0.05 radius=0.2
- added link shaft_r; visual cylinder length=0.05 radius=0.2
Joints:
- added joint shaft_l link: type fixed, parent seesaw, child shaft_l, origin xyz=0 0 0 rpy=0 0 0, axis 0.0 1.0 0.0
- added joint shaft_r link: type fixed, parent seesaw, child shaft_r, origin xyz=0 0 0 rpy=0 0 0, axis 0.0 1.0 0.0
