Commit message: modify collision of go1

File: resources/robots/go1/urdf/go1.urdf (robot description, URDF)
Before this commit: robot go1_description, 23 links, 22 joints
Links:
- added link additional_collision_box; collision box size=0.04 0.1 0.1
Joints:
- added joint head_collision: type fixed, parent base, child additional_collision_box, origin xyz=0.27 0 0 rpy=0 0 0
